File: kicad/board/scooter_board.kicad_pcb (KiCad board)
At the start: 2 copper layers, 61 x 61.2 mm, 39 parts, among them J3 Amphenol 98424-F52-12ALF, J4 OLED I2C JST-GH RA, J6 D10/SDA/SCL/5V/3V3/PACK/GND, Q1 2N7002, U2 LSM6DS3TR-C, U3 XIAO ESP32-C3

Commit message: Fix buzzer: route BZ_DRAIN to footprint pad 2
The HYG-8503A symbol mapped BZ_DRAIN to pad 3, but the buzzer's - terminal
is pad 2, so the gate drive never reached the buzzer (scope showed a clean
2.7 kHz square on the Q1 gate with nothing switching at the buzzer). Swap
the symbol's lower pin numbers 2<->3 in both the LCSC library and the
schematic's cached copy so BZ_DRAIN lands on pad 2, then update the PCB
netlist and re-route the track.

Co-Authored-By: Claude Opus 4.8 <noreply@anthropic.com>
Connections:
- BZ1 pad 2: unconnected-(BZ1-Pad2) -> BZ_DRAIN
- BZ1 pad 3: BZ_DRAIN -> unconnected-(BZ1-Pad3)
- J4 pad MP: GND -> (no net)
Routing:
- net BZ_DRAIN: track 5.60 -> 11.0 mm
- net +5V: track 115.2 -> 114.3 mm
- net GND: vias 120 -> 119
Other:
- board text added: "Turd Controller v1.1"
- board text removed: "Turd Controller v1.0"
